Commit message: Uploaded RRT Script

File: robots/youbot_with_cam3d.urdf (robot description, URDF)
Before this commit: robot youbot, 31 links, 30 joints
Links:
- added link odom
Joints:
- added joint odom_joint: type fixed, parent odom, child base_footprint, origin xyz=0 0 0 rpy=0 0 0
- joint arm_joint_2: limit lower=0 upper=2.705260340591211 effort=9.5 velocity=1.5707963267948966 -> lower=-0.75 upper=2.705260340591211 effort=9.5 velocity=1.5707963267948966
- joint arm_joint_3: limit lower=-1.0 upper=0.0 effort=9.5 velocity=1.5707963267948966 -> lower=-1.5 upper=0.0 effort=9.5 velocity=1.5707963267948966
